Commit message: Include complete laboratory world and asset rights in resources

File: laboratory_devices/centrifuge/model.urdf (robot description, URDF)
Before this commit: robot centrifuge, 3 links, 2 joints
Links:
- added link laboratory_centrifuge_lid_handle
- link laboratory_centrifuge_lid: geometry collision box size=0.014 0.016 0.086; collision box size=0.014 0.016 0.086
Joints:
- added joint laboratory_centrifuge_lid_handle_joint: type fixed, parent laboratory_centrifuge_lid, child laboratory_centrifuge_lid_handle, origin xyz=0 -0.21 0.09 rpy=0 0 0
- joint laboratory_centrifuge_lid_joint: limit lower=0 upper=1.85 effort=8 velocity=1 -> lower=0 upper=1.35 effort=8 velocity=1

File: laboratory_devices/refrigerator/model.urdf (robot description, URDF)
Before this commit: robot refrigerator, 2 links, 1 joints
Links:
- added link laboratory_refrigerator_door_handle
- link laboratory_refrigerator_door: geometry collision box size=0.016 0.035 0.016; collision box size=0.016 0.035 0.016
Joints:
- added joint laboratory_refrigerator_door_handle_joint: type fixed, parent laboratory_refrigerator_door, child laboratory_refrigerator_door_handle, origin xyz=0.482 -0.044 0 rpy=0 0 0

File: laboratory_devices/tube_rack/model.urdf (robot description, URDF)
Before this commit: robot tube_rack, 1 links, 0 joints
Links:
- added link laboratory_rack_handle
- link laboratory_rack: mass None -> 0.18; geometry collision box size=0.0023717082 0.0075025774 0.0063245553; collision box size=0.0023717082 0.0075025774 0.0063245553
Joints:
- added joint laboratory_rack_handle_joint: type fixed, parent laboratory_rack, child laboratory_rack_handle, origin xyz=0 -0.125 0.055 rpy=0 0 0
