Commit message: Update #155 Two-Sided Tote Shelving: 0.75 m clear height above the robot level (room to lift a tote clear of a robot base)
Fingerprint: two-sided tote shelving, 0 moving joints, 3 interaction frames.
Built from the WarehouseTwin asset builder (assets/shelving/build_tote_shelving.py) and exported with tools/export_to_catalogue.py.

Made with the help of Claude

File: objects_individually/storage-shelving/155-two_sided_tote_shelving/model.urdf (robot description, URDF)
Before this commit: robot two_sided_tote_shelving, 4 links, 3 joints
Joints:
- joint two_sided_tote_shelving_manual_deck_surface_fixed: origin xyz=0 0 0.8 rpy=0 0 0 -> xyz=0 0 0.95 rpy=0 0 0
