Commit message: Update #157 Mobile Tray Rack: tray in its runner (joint origin zero, geometry in the body frame), castors part of the body
Fingerprint: mobile tray rack, 1 moving joints, 4 interaction frames.
Built from the PralineTwin asset builder (assets/furnishing/build_furnishing.py) and exported with tools/export_to_catalogue.py.

Made with the help of Claude

File: objects_individually/storage-shelving/157-mobile_tray_rack/model.urdf (robot description, URDF)
Before this commit: robot mobile_tray_rack, 10 links, 9 joints
Links:
- removed link mobile_tray_rack_castor_0
- removed link mobile_tray_rack_castor_1
- removed link mobile_tray_rack_castor_2
- removed link mobile_tray_rack_castor_3
- link mobile_tray_rack_body: geometry collision box size=0.025 0.025 1.62; collision box size=0.025 0.025 1.62
Joints:
- removed joint mobile_tray_rack_castor_0_joint
- removed joint mobile_tray_rack_castor_1_joint
- removed joint mobile_tray_rack_castor_2_joint
- removed joint mobile_tray_rack_castor_3_joint
- joint mobile_tray_rack_tray_grip_fixed: origin xyz=0 -0.315 0 rpy=0 0 0 -> xyz=0 -0.315 0.95 rpy=0 0 0
- joint mobile_tray_rack_tray_joint: origin xyz=0 0 0.95 rpy=0 0 0 -> xyz=0 0 0 rpy=0 0 0
- joint mobile_tray_rack_tray_surface_fixed: origin xyz=0 0 0.006 rpy=0 0 0 -> xyz=0 0 0.956 rpy=0 0 0
